Commit message: Update leg.urdf.xacro

File: jax_ws/src/jax_description/urdf/leg.urdf.xacro (robot description, xacro)
@@ -0,0 +1,32 @@
+<?xml version="1.0"?>
+<robot xmlns:xacro="http://www.ros.org/wiki/xacro">
+  <xacro:macro name="jax_leg" params="prefix parent xyz rpy">
+    <!-- HIP -->
+    <joint name="${prefix}_hip_joint" type="revolute">
+      <parent link="${parent}"/>
+      <child link="${prefix}_hip_link"/>
+      <origin xyz="${xyz}" rpy="${rpy}"/>
+      <axis xyz="0 1 0"/>
+      <limit lower="-1.5" upper="1.5" effort="10" velocity="5"/>
+    </joint>
+    <link name="${prefix}_hip_link"/>
+    <!-- THIGH -->
+    <joint name="${prefix}_thigh_joint" type="revolute">
+      <parent link="${prefix}_hip_link"/>
+      <child link="${prefix}_thigh_link"/>
+      <origin xyz="0 0 -0.05" rpy="0 0 0"/>
+      <axis xyz="1 0 0"/>
+      <limit lower="-2.0" upper="0.5" effort="10" velocity="5"/>
+    </joint>
+    <link name="${prefix}_thigh_link"/>
+    <!-- KNEE -->
+    <joint name="${prefix}_knee_joint" type="revolute">
+      <parent link="${prefix}_thigh_link"/>
+      <child link="${prefix}_calf_link"/>
+      <origin xyz="0 0 -0.1" rpy="0 0 0"/>
+      <axis xyz="1 0 0"/>
+      <limit lower="-2.5" upper="0.0" effort="10" velocity="5"/>
+    </joint>
+    <link name="${prefix}_calf_link"/>
+  </xacro:macro>
+</robot>
