Commit message: delete

File: jax_ws/src/jax_description/urdf/jax.urdf.xacro (robot description, xacro)
@@ -0,0 +1,33 @@
+<?xml version="1.0"?>
+<robot name="jax" xmlns:xacro="http://www.ros.org/wiki/xacro">
+  <!-- ---------------- -->
+  <!-- Materials -->
+  <!-- ---------------- -->
+  <material name="black">
+    <color rgba="0.1 0.1 0.1 1.0"/>
+  </material>
+  <!-- ---------------- -->
+  <!-- Base link -->
+  <!-- ---------------- -->
+  <link name="base_link">
+    <visual>
+      <geometry>
+        <box size="0.25 0.15 0.05"/>
+      </geometry>
+      <material name="black"/>
+    </visual>
+    <collision>
+      <geometry>
+        <box size="0.25 0.15 0.05"/>
+      </geometry>
+    </collision>
+    <inertial>
+      <mass value="3.0"/>
+      <origin xyz="0 0 0"/>
+      <inertia
+        ixx="0.02" ixy="0.0" ixz="0.0"
+        iyy="0.04" iyz="0.0"
+        izz="0.05"/>
+    </inertial>
+  </link>
+</robot>

Commit message: update

File: jax_ws/src/jax_description/urdf/jax.urdf.xacro (robot description, xacro)
@@ -1,11 +1,8 @@
 <?xml version="1.0"?> <robot name="jax"
 xmlns:xacro="http://www.ros.org/wiki/xacro">
-  <!-- ---------------- --> <!--
-  Materials --> <!-- ---------------- -->
-  <material name="black">
+  <!-- Materials --> <material
+  name="black">
     <color rgba="0.1 0.1 0.1 1.0"/>
-  </material> <!-- ---------------- -->
-  <!-- Base link --> <!--
-  ---------------- --> <link
+  </material> <!-- Base link --> <link
   name="base_link">
     <visual> <geometry> <box size="0.25

Commit message: Update jax.urdf.xacro

File: jax_ws/src/jax_description/urdf/jax.urdf.xacro (robot description, xacro)
@@ -1,20 +1,30 @@
-<?xml version="1.0"?> <robot name="jax"
+<?xml version="1.0"?>
+<robot name="jax"
 xmlns:xacro="http://www.ros.org/wiki/xacro">
-  <!-- Materials --> <material
-  name="black">
+  <!-- Materials -->
+<material name="black">
     <color rgba="0.1 0.1 0.1 1.0"/>
-  </material> <!-- Base link --> <link
-  name="base_link">
-    <visual> <geometry> <box size="0.25
-        0.15 0.05"/>
-      </geometry> <material
-      name="black"/>
-    </visual> <collision> <geometry> <box
-        size="0.25 0.15 0.05"/>
-      </geometry> </collision> <inertial>
-      <mass value="3.0"/> <origin xyz="0
-      0 0"/> <inertia
+  </material>
+<!-- Base link -->
+<link name="base_link">
+    <visual>
+      <geometry>
+          <box size="0.25 0.15 0.05"/>
+      </geometry>
+      <material name="black"/>
+    </visual>
+<collision>
+  <geometry>
+    <box size="0.25 0.15 0.05"/>
+  </geometry>
+</collision>
+    <inertial>
+      <mass value="3.0"/>
+      <origin xyz="0 0 0"/>
+      <inertia
         ixx="0.02" ixy="0.0" ixz="0.0"
-        iyy="0.04" iyz="0.0" izz="0.05"/>
-    </inertial> </link>
+        iyy="0.04" iyz="0.0"
+        izz="0.05"/>
+    </inertial>
+</link>
 </robot>

Commit message: test

File: jax_ws/src/jax_description/urdf/jax.urdf.xacro (robot description, xacro)
@@ -28,3 +28,15 @@
     </inertial>
 </link>
-</robot>
+<!-- ============================= --> <!-- Front Left Hip --> <!-- ============================= --></robot> <link
+  name="front_left_hip_link">
+    <visual> <geometry> <cylinder radius="0.015" length="0.08"/> </geometry> <material name="black"/> </visual>
+    <collision>
+      <geometry> <cylinder radius="0.015" length="0.08"/> </geometry> </collision> <inertial> <mass value="0.2"/> <origin
+      xyz="0 0 0"/> <inertia
+        ixx="0.0001" ixy="0.0" ixz="0.0" iyy="0.0001" iyz="0.0" izz="0.0001"/> </inertial>
+  </link>
+<joint name="front_left_hip_joint" type="revolute"> <parent link="base_link"/> <child link="front_left_hip_link"/> <!--
+    Position relative to base --> <origin xyz="0.10 0.075 0.0" rpy="0 0 0"/> <!-- Hip rotates forward/back --> <axis
+    xyz="0 1 0"/> <limit
+      lower="-1.57" upper="1.57" effort="5.0" velocity="2.0"/>
+  </joint>

Commit message: Update jax.urdf.xacro

File: jax_ws/src/jax_description/urdf/jax.urdf.xacro (robot description, xacro)
@@ -28,15 +28,42 @@
     </inertial>
 </link>
-<!-- ============================= --> <!-- Front Left Hip --> <!-- ============================= --></robot> <link
+<!-- ============================= -->
+<!-- Front Left Hip -->
+<!-- ============================= -->
+<link
   name="front_left_hip_link">
-    <visual> <geometry> <cylinder radius="0.015" length="0.08"/> </geometry> <material name="black"/> </visual>
-    <collision>
-      <geometry> <cylinder radius="0.015" length="0.08"/> </geometry> </collision> <inertial> <mass value="0.2"/> <origin
-      xyz="0 0 0"/> <inertia
-        ixx="0.0001" ixy="0.0" ixz="0.0" iyy="0.0001" iyz="0.0" izz="0.0001"/> </inertial>
-  </link>
-<joint name="front_left_hip_joint" type="revolute"> <parent link="base_link"/> <child link="front_left_hip_link"/> <!--
-    Position relative to base --> <origin xyz="0.10 0.075 0.0" rpy="0 0 0"/> <!-- Hip rotates forward/back --> <axis
-    xyz="0 1 0"/> <limit
-      lower="-1.57" upper="1.57" effort="5.0" velocity="2.0"/>
+    <visual>
+      <geometry>
+        <cylinder radius="0.015" length="0.08"/>
+      </geometry>
+      <material name="black"/>
+    </visual>
+<collision>
+      <geometry>
+        <cylinder radius="0.015" length="0.08"/>
+        </geometry>
+</collision>
+<inertial>
+<mass value="0.2"/>
+<origin xyz="0 0 0"/>
+<inertia
+      ixx="0.0001" ixy="0.0" ixz="0.0"
+      iyy="0.0001" iyz="0.0"
+      izz="0.0001"/>
+</inertial>
+</link>
+<joint name="front_left_hip_joint"
+type="revolute">
+  <parent link="base_link"/>
+  <child link="front_left_hip_link"/>
+<!--Position relative to base -->
+<origin xyz="0.10 0.075 0.0" rpy="0 0 0"/>
+<!-- Hip rotates forward/back -->
+<axis xyz="0 1 0"/>
+<limit
+      lower="-1.57"
+      upper="1.57"
+      effort="5.0"
+      velocity="2.0"/>
   </joint>
+</robot>

Commit message: added

File: jax_ws/src/jax_description/urdf/jax.urdf.xacro (robot description, xacro)
@@ -2,4 +2,12 @@
 <robot name="jax"
 xmlns:xacro="http://www.ros.org/wiki/xacro">
+  <!-- World link -->
+  <link name="world"/>
+  <!-- Fixed joint to base -->
+  <joint name="world_to_base" type="fixed">
+    <parent link="world"/>
+    <child link="base_link"/>
+    <origin xyz="0 0 0" rpy="0 0 0"/>
+  </joint>
   <!-- Materials -->
 <material name="black">

Commit message: adding leg

File: jax_ws/src/jax_description/urdf/jax.urdf.xacro (robot description, xacro)
@@ -36,4 +36,48 @@
     </inertial>
 </link>
+  <!-- FRONT LEFT LEG -->
+  <link name="front_left_hip">
+    <visual>
+      <geometry>
+        <cylinder length="0.05" radius="0.02"/>
+      </geometry>
+      <material name="black"/>
+    </visual>
+  </link>
+  <joint name="front_left_hip_joint" type="revolute">
+    <parent link="base_link"/>
+    <child link="front_left_hip"/>
+    <origin xyz="0.12 0.08 0.0"/>
+    <axis xyz="0 1 0"/>
+    <limit lower="-1.57" upper="1.57" effort="1.0" velocity="1.0"/>
+  </joint>
+  <link name="front_left_thigh">
+    <visual>
+      <geometry>
+        <cylinder length="0.12" radius="0.015"/>
+      </geometry>
+    </visual>
+  </link>
+  <joint name="front_left_thigh_joint" type="revolute">
+    <parent link="front_left_hip"/>
+    <child link="front_left_thigh"/>
+    <origin xyz="0 0 -0.06"/>
+    <axis xyz="1 0 0"/>
+    <limit lower="-1.57" upper="1.57" effort="1.0" velocity="1.0"/>
+  </joint>
+  <link name="front_left_calf">
+    <visual>
+      <geometry>
+        <cylinder length="0.12" radius="0.012"/>
+      </geometry>
+    </visual>
+  </link>
+  <joint name="front_left_knee_joint" type="revolute">
+    <parent link="front_left_thigh"/>
+    <child link="front_left_calf"/>
+    <origin xyz="0 0 -0.12"/>
+    <axis xyz="1 0 0"/>
+    <limit lower="-1.57" upper="1.57" effort="1.0" velocity="1.0"/>
+  </joint>
 <!-- ============================= -->
 <!-- Front Left Hip -->

Commit message: fix

File: jax_ws/src/jax_description/urdf/jax.urdf.xacro (robot description, xacro)
@@ -80,42 +80,3 @@
     <limit lower="-1.57" upper="1.57" effort="1.0" velocity="1.0"/>
   </joint>
-<!-- ============================= -->
-<!-- Front Left Hip -->
-<!-- ============================= -->
-<link
-  name="front_left_hip_link">
-    <visual>
-      <geometry>
-        <cylinder radius="0.015" length="0.08"/>
-      </geometry>
-      <material name="black"/>
-    </visual>
-<collision>
-      <geometry>
-        <cylinder radius="0.015" length="0.08"/>
-        </geometry>
-</collision>
-<inertial>
-<mass value="0.2"/>
-<origin xyz="0 0 0"/>
-<inertia
-      ixx="0.0001" ixy="0.0" ixz="0.0"
-      iyy="0.0001" iyz="0.0"
-      izz="0.0001"/>
-</inertial>
-</link>
-<joint name="front_left_hip_joint"
-type="revolute">
-  <parent link="base_link"/>
-  <child link="front_left_hip_link"/>
-<!--Position relative to base -->
-<origin xyz="0.10 0.075 0.0" rpy="0 0 0"/>
-<!-- Hip rotates forward/back -->
-<axis xyz="0 1 0"/>
-<limit
-      lower="-1.57"
-      upper="1.57"
-      effort="5.0"
-      velocity="2.0"/>
-  </joint>
 </robot>

Commit message: added right leg

File: jax_ws/src/jax_description/urdf/jax.urdf.xacro (robot description, xacro)
@@ -80,3 +80,47 @@
     <limit lower="-1.57" upper="1.57" effort="1.0" velocity="1.0"/>
   </joint>
+  <!-- FRONT RIGHT LEG -->
+  <link name="front_right_hip">
+    <visual>
+      <geometry>
+        <cylinder length="0.05" radius="0.02"/>
+      </geometry>
+      <material name="black"/>
+    </visual>
+  </link>
+  <joint name="front_right_hip_joint" type="revolute">
+    <parent link="base_link"/>
+    <child link="front_right_hip"/>
+    <origin xyz="0.12 -0.08 0.0"/>
+    <axis xyz="0 -1 0"/>
+    <limit lower="-1.57" upper="1.57" effort="1.0" velocity="1.0"/>
+  </joint>
+  <link name="front_right_thigh">
+    <visual>
+      <geometry>
+        <cylinder length="0.12" radius="0.015"/>
+      </geometry>
+    </visual>
+  </link>
+  <joint name="front_right_thigh_joint" type="revolute">
+    <parent link="front_right_hip"/>
+    <child link="front_right_thigh"/>
+    <origin xyz="0 0 -0.06"/>
+    <axis xyz="0 -1 0"/>
+    <limit lower="-1.57" upper="1.57" effort="1.0" velocity="1.0"/>
+  </joint>
+  <link name="front_right_calf">
+    <visual>
+      <geometry>
+        <cylinder length="0.12" radius="0.012"/>
+      </geometry>
+    </visual>
+  </link>
+  <joint name="front_right_knee_joint" type="revolute">
+    <parent link="front_right_thigh"/>
+    <child link="front_right_calf"/>
+    <origin xyz="0 0 -0.12"/>
+    <axis xyz="0 -1 0"/>
+    <limit lower="-1.57" upper="1.57" effort="1.0" velocity="1.0"/>
+  </joint>
 </robot>

Commit message: fix axis

File: jax_ws/src/jax_description/urdf/jax.urdf.xacro (robot description, xacro)
@@ -63,5 +63,5 @@
     <child link="front_left_thigh"/>
     <origin xyz="0 0 -0.06"/>
-    <axis xyz="1 0 0"/>
+    <axis xyz="0 1 0"/>
     <limit lower="-1.57" upper="1.57" effort="1.0" velocity="1.0"/>
   </joint>
@@ -77,5 +77,5 @@
     <child link="front_left_calf"/>
     <origin xyz="0 0 -0.12"/>
-    <axis xyz="1 0 0"/>
+    <axis xyz="0 1 0"/>
     <limit lower="-1.57" upper="1.57" effort="1.0" velocity="1.0"/>
   </joint>

Commit message: fix hip

File: jax_ws/src/jax_description/urdf/jax.urdf.xacro (robot description, xacro)
@@ -49,5 +49,5 @@
     <child link="front_left_hip"/>
     <origin xyz="0.12 0.08 0.0"/>
-    <axis xyz="0 1 0"/>
+    <axis xyz="0 0 1"/>
     <limit lower="-1.57" upper="1.57" effort="1.0" velocity="1.0"/>
   </joint>
@@ -93,5 +93,5 @@
     <child link="front_right_hip"/>
     <origin xyz="0.12 -0.08 0.0"/>
-    <axis xyz="0 -1 0"/>
+    <axis xyz="0 0 -1"/>
     <limit lower="-1.57" upper="1.57" effort="1.0" velocity="1.0"/>
   </joint>

Commit message: fix

File: jax_ws/src/jax_description/urdf/jax.urdf.xacro (robot description, xacro)
@@ -68,4 +68,5 @@
   <link name="front_left_calf">
     <visual>
+      <origin xyz="0 0 -0.06"/>
       <geometry>
         <cylinder length="0.12" radius="0.012"/>
@@ -76,5 +77,5 @@
     <parent link="front_left_thigh"/>
     <child link="front_left_calf"/>
-    <origin xyz="0 0 -0.12"/>
+    <origin xyz="0 0 0"/>
     <axis xyz="0 1 0"/>
     <limit lower="-1.57" upper="1.57" effort="1.0" velocity="1.0"/>
@@ -112,4 +113,5 @@
   <link name="front_right_calf">
     <visual>
+      <origin xyz="0 0 -0.06"/>
       <geometry>
         <cylinder length="0.12" radius="0.012"/>
@@ -120,5 +122,5 @@
     <parent link="front_right_thigh"/>
     <child link="front_right_calf"/>
-    <origin xyz="0 0 -0.12"/>
+    <origin xyz="0 0 0"/>
     <axis xyz="0 -1 0"/>
     <limit lower="-1.57" upper="1.57" effort="1.0" velocity="1.0"/>

Commit message: fix

File: jax_ws/src/jax_description/urdf/jax.urdf.xacro (robot description, xacro)
@@ -90,11 +90,11 @@
     </visual>
   </link>
-  <joint name="front_right_hip_joint" type="revolute">
-    <parent link="base_link"/>
-    <child link="front_right_hip"/>
-    <origin xyz="0.12 -0.08 0.0"/>
-    <axis xyz="0 0 -1"/>
-    <limit lower="-1.57" upper="1.57" effort="1.0" velocity="1.0"/>
-  </joint>
+<joint name="front_right_hip_joint" type="prismatic">
+  <parent link="base_link"/>
+  <child link="front_right_hip"/>
+  <origin xyz="0.12 -0.08 0.0"/>
+  <axis xyz="0 -1 0"/>
+  <limit lower="-0.03" upper="0.03" effort="1.0" velocity="0.1"/>
+</joint>
   <link name="front_right_thigh">
     <visual>

Commit message: fix

File: jax_ws/src/jax_description/urdf/jax.urdf.xacro (robot description, xacro)
@@ -90,10 +90,10 @@
     </visual>
   </link>
-<joint name="front_right_hip_joint" type="prismatic">
+<joint name="front_right_hip_joint" type="revolute">
   <parent link="base_link"/>
   <child link="front_right_hip"/>
   <origin xyz="0.12 -0.08 0.0"/>
-  <axis xyz="0 -1 0"/>
-  <limit lower="-0.03" upper="0.03" effort="1.0" velocity="0.1"/>
+  <axis xyz="1 0 0"/>
+  <limit lower="-0.6" upper="0.6" effort="1.0" velocity="1.0"/>
 </joint>
   <link name="front_right_thigh">

Commit message: fix

File: jax_ws/src/jax_description/urdf/jax.urdf.xacro (robot description, xacro)
@@ -97,15 +97,16 @@
   <limit lower="-0.6" upper="0.6" effort="1.0" velocity="1.0"/>
 </joint>
-  <link name="front_right_thigh">
-    <visual>
-      <geometry>
-        <cylinder length="0.12" radius="0.015"/>
-      </geometry>
-    </visual>
-  </link>
+<link name="front_right_thigh">
+  <visual>
+    <origin xyz="0 0 -0.06"/>
+    <geometry>
+      <cylinder length="0.12" radius="0.015"/>
+    </geometry>
+  </visual>
+</link>
   <joint name="front_right_thigh_joint" type="revolute">
     <parent link="front_right_hip"/>
     <child link="front_right_thigh"/>
-    <origin xyz="0 0 -0.06"/>
+    <origin xyz="0 0 0"/>
     <axis xyz="0 -1 0"/>
     <limit lower="-1.57" upper="1.57" effort="1.0" velocity="1.0"/>

Commit message: fix

File: jax_ws/src/jax_description/urdf/jax.urdf.xacro (robot description, xacro)
@@ -114,5 +114,5 @@
   <link name="front_right_calf">
     <visual>
-      <origin xyz="0 0 -0.06"/>
+      <origin xyz="0 0 -0.12"/>
       <geometry>
         <cylinder length="0.12" radius="0.012"/>

Commit message: fix

File: jax_ws/src/jax_description/urdf/jax.urdf.xacro (robot description, xacro)
@@ -114,5 +114,5 @@
   <link name="front_right_calf">
     <visual>
-      <origin xyz="0 0 -0.12"/>
+      <origin xyz="0 0 -0.06"/>
       <geometry>
         <cylinder length="0.12" radius="0.012"/>

Commit message: c

File: jax_ws/src/jax_description/urdf/jax.urdf.xacro (robot description, xacro)
@@ -114,5 +114,5 @@
   <link name="front_right_calf">
     <visual>
-      <origin xyz="0 0 -0.12"/>
+      <origin xyz="0 0 -0.18"/>
       <geometry>
         <cylinder length="0.12" radius="0.012"/>

Commit message: d

File: jax_ws/src/jax_description/urdf/jax.urdf.xacro (robot description, xacro)
@@ -123,5 +123,5 @@
     <parent link="front_right_thigh"/>
     <child link="front_right_calf"/>
-    <origin xyz="0 0 0"/>
+    <origin xyz="0 0 -0.06"/>
     <axis xyz="0 -1 0"/>
     <limit lower="-1.57" upper="1.57" effort="1.0" velocity="1.0"/>

Commit message: d

File: jax_ws/src/jax_description/urdf/jax.urdf.xacro (robot description, xacro)
@@ -114,5 +114,5 @@
   <link name="front_right_calf">
     <visual>
-      <origin xyz="0 0 -0.18"/>
+      <origin xyz="0 0 -0.6"/>
       <geometry>
         <cylinder length="0.12" radius="0.012"/>
@@ -121,9 +121,9 @@
   </link>
   <joint name="front_right_knee_joint" type="revolute">
-    <parent link="front_right_thigh"/>
-    <child link="front_right_calf"/>
-    <origin xyz="0 0 -0.06"/>
-    <axis xyz="0 -1 0"/>
-    <limit lower="-1.57" upper="1.57" effort="1.0" velocity="1.0"/>
-  </joint>
+  <parent link="front_right_thigh"/>
+  <child link="front_right_calf"/>
+  <origin xyz="0 0 -0.12"/>
+  <axis xyz="0 -1 0"/>
+  <limit lower="-1.57" upper="1.57" effort="1.0" velocity="1.0"/>
+</joint>
 </robot>

Commit message: d

File: jax_ws/src/jax_description/urdf/jax.urdf.xacro (robot description, xacro)
@@ -123,5 +123,5 @@
   <parent link="front_right_thigh"/>
   <child link="front_right_calf"/>
-  <origin xyz="0 0 -0.12"/>
+  <origin xyz="0 0 0"/>
   <axis xyz="0 -1 0"/>
   <limit lower="-1.57" upper="1.57" effort="1.0" velocity="1.0"/>

Commit message: d

File: jax_ws/src/jax_description/urdf/jax.urdf.xacro (robot description, xacro)
@@ -114,9 +114,9 @@
   <link name="front_right_calf">
     <visual>
-      <origin xyz="0 0 -0.6"/>
+      <origin xyz="0 0 0"/>
       <geometry>
         <cylinder length="0.12" radius="0.012"/>
       </geometry>
-    </visual>
+    </visual>d
   </link>
   <joint name="front_right_knee_joint" type="revolute">

Commit message: f

File: jax_ws/src/jax_description/urdf/jax.urdf.xacro (robot description, xacro)
@@ -114,5 +114,5 @@
   <link name="front_right_calf">
     <visual>
-      <origin xyz="0 0 0"/>
+      <origin xyz="0 0 -0.06"/>
       <geometry>
         <cylinder length="0.12" radius="0.012"/>

Commit message: f

File: jax_ws/src/jax_description/urdf/jax.urdf.xacro (robot description, xacro)
@@ -99,5 +99,5 @@
 <link name="front_right_thigh">
   <visual>
-    <origin xyz="0 0 -0.06"/>
+    <origin xyz="0 0 0.06"/>
     <geometry>
       <cylinder length="0.12" radius="0.015"/>

Commit message: d

File: jax_ws/src/jax_description/urdf/jax.urdf.xacro (robot description, xacro)
@@ -108,5 +108,5 @@
     <parent link="front_right_hip"/>
     <child link="front_right_thigh"/>
-    <origin xyz="0 0 0"/>
+    <origin xyz="0 0 -0.06"/>
     <axis xyz="0 -1 0"/>
     <limit lower="-1.57" upper="1.57" effort="1.0" velocity="1.0"/>

Commit message: f

File: jax_ws/src/jax_description/urdf/jax.urdf.xacro (robot description, xacro)
@@ -108,5 +108,5 @@
     <parent link="front_right_hip"/>
     <child link="front_right_thigh"/>
-    <origin xyz="0 0 -0.06"/>
+    <origin xyz="0 0 0"/>
     <axis xyz="0 -1 0"/>
     <limit lower="-1.57" upper="1.57" effort="1.0" velocity="1.0"/>

Commit message: f

File: jax_ws/src/jax_description/urdf/jax.urdf.xacro (robot description, xacro)
@@ -99,5 +99,5 @@
 <link name="front_right_thigh">
   <visual>
-    <origin xyz="0 0 0.06"/>
+    <origin xyz="0 0 0"/>
     <geometry>
       <cylinder length="0.12" radius="0.015"/>

Commit message: d

File: jax_ws/src/jax_description/urdf/jax.urdf.xacro (robot description, xacro)
@@ -99,5 +99,5 @@
 <link name="front_right_thigh">
   <visual>
-    <origin xyz="0 0 0"/>
+    <origin xyz="0 0 -0.06"/>
     <geometry>
       <cylinder length="0.12" radius="0.015"/>
@@ -114,5 +114,5 @@
   <link name="front_right_calf">
     <visual>
-      <origin xyz="0 0 -0.06"/>
+      <origin xyz="0 0 -0.12"/>
       <geometry>
         <cylinder length="0.12" radius="0.012"/>

Commit message: d

File: jax_ws/src/jax_description/urdf/jax.urdf.xacro (robot description, xacro)
@@ -123,5 +123,5 @@
   <parent link="front_right_thigh"/>
   <child link="front_right_calf"/>
-  <origin xyz="0 0 0"/>
+  <origin xyz="0 0 -0.06"/>
   <axis xyz="0 -1 0"/>
   <limit lower="-1.57" upper="1.57" effort="1.0" velocity="1.0"/>

Commit message: f

File: jax_ws/src/jax_description/urdf/jax.urdf.xacro (robot description, xacro)
@@ -123,5 +123,5 @@
   <parent link="front_right_thigh"/>
   <child link="front_right_calf"/>
-  <origin xyz="0 0 -0.06"/>
+  <origin xyz="0 0 0"/>
   <axis xyz="0 -1 0"/>
   <limit lower="-1.57" upper="1.57" effort="1.0" velocity="1.0"/>

Commit message: ddd

File: jax_ws/src/jax_description/urdf/jax.urdf.xacro (robot description, xacro)
@@ -114,5 +114,5 @@
   <link name="front_right_calf">
     <visual>
-      <origin xyz="0 0 -0.06"/>
+      <origin xyz="0 0 -0.18"/>
       <geometry>
         <cylinder length="0.12" radius="0.012"/>

Commit message: d

File: jax_ws/src/jax_description/urdf/jax.urdf.xacro (robot description, xacro)
@@ -123,5 +123,5 @@
   <parent link="front_right_thigh"/>
   <child link="front_right_calf"/>
-  <origin xyz="0 0 0"/>
+  <origin xyz="0 0 -0.12"/>
   <axis xyz="0 -1 0"/>
   <limit lower="-1.57" upper="1.57" effort="1.0" velocity="1.0"/>

Commit message: ff

File: jax_ws/src/jax_description/urdf/jax.urdf.xacro (robot description, xacro)
@@ -114,5 +114,5 @@
   <link name="front_right_calf">
     <visual>
-      <origin xyz="0 0 -0.18"/>
+      <origin xyz="0 0 -0.06"/>
       <geometry>
         <cylinder length="0.12" radius="0.012"/>
@@ -123,5 +123,5 @@
   <parent link="front_right_thigh"/>
   <child link="front_right_calf"/>
-  <origin xyz="0 0 0"/>
+  <origin xyz="0 0 -0.12"/>
   <axis xyz="0 -1 0"/>
   <limit lower="-1.57" upper="1.57" effort="1.0" velocity="1.0"/>
