Commit message: left leg

File: jax_ws/src/jax_description/urdf/jax.urdf.xacro (robot description, xacro)
@@ -36,49 +36,4 @@
     </inertial>
 </link>
-  <!-- FRONT LEFT LEG -->
-  <link name="front_left_hip">
-    <visual>
-      <geometry>
-        <cylinder length="0.05" radius="0.02"/>
-      </geometry>
-      <material name="black"/>
-    </visual>
-  </link>
-  <joint name="front_left_hip_joint" type="revolute">
-    <parent link="base_link"/>
-    <child link="front_left_hip"/>
-    <origin xyz="0.12 0.08 0.0"/>
-    <axis xyz="0 0 1"/>
-    <limit lower="-1.57" upper="1.57" effort="1.0" velocity="1.0"/>
-  </joint>
-  <link name="front_left_thigh">
-    <visual>
-      <geometry>
-        <cylinder length="0.12" radius="0.015"/>
-      </geometry>
-    </visual>
-  </link>
-  <joint name="front_left_thigh_joint" type="revolute">
-    <parent link="front_left_hip"/>
-    <child link="front_left_thigh"/>
-    <origin xyz="0 0 -0.06"/>
-    <axis xyz="0 1 0"/>
-    <limit lower="-1.57" upper="1.57" effort="1.0" velocity="1.0"/>
-  </joint>
-  <link name="front_left_calf">
-    <visual>
-      <origin xyz="0 0 -0.06"/>
-      <geometry>
-        <cylinder length="0.12" radius="0.012"/>
-      </geometry>
-    </visual>
-  </link>
-  <joint name="front_left_knee_joint" type="revolute">
-    <parent link="front_left_thigh"/>
-    <child link="front_left_calf"/>
-    <origin xyz="0 0 0"/>
-    <axis xyz="0 1 0"/>
-    <limit lower="-1.57" upper="1.57" effort="1.0" velocity="1.0"/>
-  </joint>
   <!-- FRONT RIGHT LEG -->
   <link name="front_right_hip">
@@ -118,6 +73,6 @@
         <cylinder length="0.12" radius="0.012"/>
       </geometry>
-    </visual>d
-  </link>
+    </visual>
+   </link>
   <joint name="front_right_knee_joint" type="revolute">
   <parent link="front_right_thigh"/>
@@ -127,3 +82,49 @@
   <limit lower="-1.57" upper="1.57" effort="1.0" velocity="1.0"/>
 </joint>
+<!-- FRONT LEFT LEG -->
+<link name="front_left_hip">
+  <visual>
+    <geometry>
+      <cylinder length="0.05" radius="0.02"/>
+    </geometry>
+    <material name="black"/>
+  </visual>
+</link>
+<joint name="front_left_hip_joint" type="revolute">
+  <parent link="base_link"/>
+  <child link="front_left_hip"/>
+  <origin xyz="0.12 0.08 0.0"/>
+  <axis xyz="1 0 0"/>
+  <limit lower="-0.6" upper="0.6" effort="1.0" velocity="1.0"/>
+</joint>
+<link name="front_left_thigh">
+  <visual>
+    <origin xyz="0 0 -0.06"/>
+    <geometry>
+      <cylinder length="0.12" radius="0.015"/>
+    </geometry>
+  </visual>
+</link>
+<joint name="front_left_thigh_joint" type="revolute">
+  <parent link="front_left_hip"/>
+  <child link="front_left_thigh"/>
+  <origin xyz="0 0 0"/>
+  <axis xyz="0 1 0"/>
+  <limit lower="-1.57" upper="1.57" effort="1.0" velocity="1.0"/>
+</joint>
+<link name="front_left_calf">
+  <visual>
+    <origin xyz="0 0 -0.06"/>
+    <geometry>
+      <cylinder length="0.12" radius="0.012"/>
+    </geometry>
+  </visual>
+</link>
+<joint name="front_left_knee_joint" type="revolute">
+  <parent link="front_left_thigh"/>
+  <child link="front_left_calf"/>
+  <origin xyz="0 0 -0.12"/>
+  <axis xyz="0 1 0"/>
+  <limit lower="-1.57" upper="1.57" effort="1.0" velocity="1.0"/>
+</joint>
 </robot>

Commit message: rear right

File: jax_ws/src/jax_description/urdf/jax.urdf.xacro (robot description, xacro)
@@ -128,3 +128,49 @@
   <limit lower="-1.57" upper="1.57" effort="1.0" velocity="1.0"/>
 </joint>
+<!-- REAR RIGHT LEG -->
+<link name="rear_right_hip">
+  <visual>
+    <geometry>
+      <cylinder length="0.05" radius="0.02"/>
+    </geometry>
+    <material name="black"/>
+  </visual>
+</link>
+<joint name="rear_right_hip_joint" type="revolute">
+  <parent link="base_link"/>
+  <child link="rear_right_hip"/>
+  <origin xyz="-0.12 -0.08 0.0"/>
+  <axis xyz="1 0 0"/>
+  <limit lower="-0.6" upper="0.6" effort="1.0" velocity="1.0"/>
+</joint>
+<link name="rear_right_thigh">
+  <visual>
+    <origin xyz="0 0 -0.06"/>
+    <geometry>
+      <cylinder length="0.12" radius="0.015"/>
+    </geometry>
+  </visual>
+</link>
+<joint name="rear_right_thigh_joint" type="revolute">
+  <parent link="rear_right_hip"/>
+  <child link="rear_right_thigh"/>
+  <origin xyz="0 0 0"/>
+  <axis xyz="0 -1 0"/>
+  <limit lower="-1.57" upper="1.57" effort="1.0" velocity="1.0"/>
+</joint>
+<link name="rear_right_calf">
+  <visual>
+    <origin xyz="0 0 -0.06"/>
+    <geometry>
+      <cylinder length="0.12" radius="0.012"/>
+    </geometry>
+  </visual>
+</link>
+<joint name="rear_right_knee_joint" type="revolute">
+  <parent link="rear_right_thigh"/>
+  <child link="rear_right_calf"/>
+  <origin xyz="0 0 -0.12"/>
+  <axis xyz="0 -1 0"/>
+  <limit lower="-1.57" upper="1.57" effort="1.0" velocity="1.0"/>
+</joint>
 </robot>

Commit message: rear left

File: jax_ws/src/jax_description/urdf/jax.urdf.xacro (robot description, xacro)
@@ -174,3 +174,49 @@
   <limit lower="-1.57" upper="1.57" effort="1.0" velocity="1.0"/>
 </joint>
+<!-- REAR LEFT LEG -->
+<link name="rear_left_hip">
+  <visual>
+    <geometry>
+      <cylinder length="0.05" radius="0.02"/>
+    </geometry>
+    <material name="black"/>
+  </visual>
+</link>
+<joint name="rear_left_hip_joint" type="revolute">
+  <parent link="base_link"/>
+  <child link="rear_left_hip"/>
+  <origin xyz="-0.12 0.08 0.0"/>
+  <axis xyz="1 0 0"/>
+  <limit lower="-0.6" upper="0.6" effort="1.0" velocity="1.0"/>
+</joint>
+<link name="rear_left_thigh">
+  <visual>
+    <origin xyz="0 0 -0.06"/>
+    <geometry>
+      <cylinder length="0.12" radius="0.015"/>
+    </geometry>
+  </visual>
+</link>
+<joint name="rear_left_thigh_joint" type="revolute">
+  <parent link="rear_left_hip"/>
+  <child link="rear_left_thigh"/>
+  <origin xyz="0 0 0"/>
+  <axis xyz="0 1 0"/>
+  <limit lower="-1.57" upper="1.57" effort="1.0" velocity="1.0"/>
+</joint>
+<link name="rear_left_calf">
+  <visual>
+    <origin xyz="0 0 -0.06"/>
+    <geometry>
+      <cylinder length="0.12" radius="0.012"/>
+    </geometry>
+  </visual>
+</link>
+<joint name="rear_left_knee_joint" type="revolute">
+  <parent link="rear_left_thigh"/>
+  <child link="rear_left_calf"/>
+  <origin xyz="0 0 -0.12"/>
+  <axis xyz="0 1 0"/>
+  <limit lower="-1.57" upper="1.57" effort="1.0" velocity="1.0"/>
+</joint>
 </robot>

Commit message: fix knee joint

File: jax_ws/src/jax_description/urdf/jax.urdf.xacro (robot description, xacro)
@@ -80,5 +80,5 @@
   <origin xyz="0 0 -0.12"/>
   <axis xyz="0 -1 0"/>
-  <limit lower="-1.57" upper="1.57" effort="1.0" velocity="1.0"/>
+  <limit lower="0.0" upper="1.57" effort="1.0" velocity="1.0"/>
 </joint>
 <!-- FRONT LEFT LEG -->
@@ -126,5 +126,5 @@
   <origin xyz="0 0 -0.12"/>
   <axis xyz="0 1 0"/>
-  <limit lower="-1.57" upper="1.57" effort="1.0" velocity="1.0"/>
+  <limit lower="0.0" upper="1.57" effort="1.0" velocity="1.0"/>
 </joint>
 <!-- REAR RIGHT LEG -->
@@ -172,5 +172,5 @@
   <origin xyz="0 0 -0.12"/>
   <axis xyz="0 -1 0"/>
-  <limit lower="-1.57" upper="1.57" effort="1.0" velocity="1.0"/>
+  <limit lower="0.0" upper="1.57" effort="1.0" velocity="1.0"/>
 </joint>
 <!-- REAR LEFT LEG -->
@@ -218,5 +218,5 @@
   <origin xyz="0 0 -0.12"/>
   <axis xyz="0 1 0"/>
-  <limit lower="-1.57" upper="1.57" effort="1.0" velocity="1.0"/>
+  <limit lower="0.0" upper="1.57" effort="1.0" velocity="1.0"/>
 </joint>
 </robot>

Commit message: fix

File: jax_ws/src/jax_description/urdf/jax.urdf.xacro (robot description, xacro)
@@ -79,5 +79,5 @@
   <child link="front_right_calf"/>
   <origin xyz="0 0 -0.12"/>
-  <axis xyz="0 -1 0"/>
+  <axis xyz="0 1 0"/>
   <limit lower="0.0" upper="1.57" effort="1.0" velocity="1.0"/>
 </joint>
@@ -125,5 +125,5 @@
   <child link="front_left_calf"/>
   <origin xyz="0 0 -0.12"/>
-  <axis xyz="0 1 0"/>
+  <axis xyz="0 -1 0"/>
   <limit lower="0.0" upper="1.57" effort="1.0" velocity="1.0"/>
 </joint>
@@ -171,5 +171,5 @@
   <child link="rear_right_calf"/>
   <origin xyz="0 0 -0.12"/>
-  <axis xyz="0 -1 0"/>
+  <axis xyz="0 1 0"/>
   <limit lower="0.0" upper="1.57" effort="1.0" velocity="1.0"/>
 </joint>
@@ -217,5 +217,5 @@
   <child link="rear_left_calf"/>
   <origin xyz="0 0 -0.12"/>
-  <axis xyz="0 1 0"/>
+  <axis xyz="0 -1 0"/>
   <limit lower="0.0" upper="1.57" effort="1.0" velocity="1.0"/>
 </joint>

Commit message: f

File: jax_ws/src/jax_description/urdf/jax.urdf.xacro (robot description, xacro)
@@ -125,5 +125,5 @@
   <child link="front_left_calf"/>
   <origin xyz="0 0 -0.12"/>
-  <axis xyz="0 -1 0"/>
+  <axis xyz="0 1 0"/>
   <limit lower="0.0" upper="1.57" effort="1.0" velocity="1.0"/>
 </joint>
@@ -217,5 +217,5 @@
   <child link="rear_left_calf"/>
   <origin xyz="0 0 -0.12"/>
-  <axis xyz="0 -1 0"/>
+  <axis xyz="0 1 0"/>
   <limit lower="0.0" upper="1.57" effort="1.0" velocity="1.0"/>
 </joint>

Commit message: Update jax.urdf.xacro

File: jax_ws/src/jax_description/urdf/jax.urdf.xacro (robot description, xacro)
@@ -56,5 +56,7 @@
     <origin xyz="0 0 -0.06"/>
     <geometry>
-      <cylinder length="0.12" radius="0.015"/>
+      <mesh filename="package://jax_description/meshes/front_right_thigh.stl"
+          scale="1 1 1"/>
+      # <cylinder length="0.12" radius="0.015"/>
     </geometry>
   </visual>

Commit message: Update jax.urdf.xacro

File: jax_ws/src/jax_description/urdf/jax.urdf.xacro (robot description, xacro)
@@ -58,5 +58,5 @@
       <mesh filename="package://jax_description/meshes/front_right_thigh.stl"
           scale="1 1 1"/>
-      # <cylinder length="0.12" radius="0.015"/>
+       <!-- <cylinder length="0.12" radius="0.015"/> -->
     </geometry>
   </visual>

Commit message: Update jax.urdf.xacro

File: jax_ws/src/jax_description/urdf/jax.urdf.xacro (robot description, xacro)
@@ -56,8 +56,6 @@
     <origin xyz="0 0 -0.06"/>
     <geometry>
-      <mesh filename="package://jax_description/meshes/front_right_thigh.stl"
-          scale="1 1 1"/>
-       <!-- <cylinder length="0.12" radius="0.015"/> -->
-    </geometry>
+         <cylinder length="0.12" radius="0.015"/>
+  </geometry>
   </visual>
 </link>

Commit message: adding mesh

File: jax_ws/src/jax_description/urdf/jax.urdf.xacro (robot description, xacro)
@@ -16,24 +16,27 @@
 <!-- Base link -->
 <link name="base_link">
-    <visual>
-      <geometry>
-          <box size="0.25 0.15 0.05"/>
-      </geometry>
-      <material name="black"/>
-    </visual>
-<collision>
+  <visual>
+  <origin xyz="0 0 0" rpy="0 0 0"/>
   <geometry>
     <mesh filename="package://jax_description/meshes/base_link.stl"
-            scale="0.001 0.001 0.001"/>
+          scale="1 1 1"/>
+  </geometry>
+  <material name="black"/>
+</visual>
+<collision>
+  <origin xyz="0 0 0" rpy="0 0 0"/>
+  <geometry>
+    <mesh filename="package://jax_description/meshes/base_collision.stl"
+          scale="1 1 1"/>
   </geometry>
 </collision>
-    <inertial>
-      <mass value="3.0"/>
-      <origin xyz="0 0 0"/>
-      <inertia
-        ixx="0.02" ixy="0.0" ixz="0.0"
-        iyy="0.04" iyz="0.0"
-        izz="0.05"/>
-    </inertial>
+  <inertial>
+    <mass value="3.0"/>
+    <origin xyz="0 0 0"/>
+    <inertia
+      ixx="0.02" ixy="0.0" ixz="0.0"
+      iyy="0.04" iyz="0.0"
+      izz="0.05"/>
+  </inertial>
 </link>
   <!-- FRONT RIGHT LEG -->
@@ -55,7 +58,8 @@
 <link name="front_right_thigh">
   <visual>
-    <origin xyz="0 0 -0.06"/>
-    <geometry>
-         <cylinder length="0.12" radius="0.015"/>
+    <origin xyz="0 0 0" rpy="1.5708 1.5708 0"/>
+    <geometry>
+          <mesh filename="package://jax_description/meshes/front_right_thigh.stl"
+          scale="1 1 1"/>
   </geometry>
   </visual>

Commit message: dd

File: jax_ws/src/jax_description/urdf/jax.urdf.xacro (robot description, xacro)
@@ -14,4 +14,7 @@
     <color rgba="0.1 0.1 0.1 1.0"/>
   </material>
+  <material name="white">
+  <color rgba="1 1 1 1"/>
+</material>
 <!-- Base link -->
 <link name="base_link">
@@ -43,8 +46,10 @@
   <link name="front_right_hip">
     <visual>
+      <origin xyz="-0.01 0.02 -0.015" rpy="-1.5708 3.1416 -1.5708"/>
       <geometry>
-        <cylinder length="0.05" radius="0.02"/>
+        <mesh filename="package://jax_description/meshes/front_right_hip.stl"
+          scale="1 1 1"/>
       </geometry>
-      <material name="black"/>
+      <material name="white"/>
     </visual>
   </link>
@@ -58,5 +63,5 @@
 <link name="front_right_thigh">
   <visual>
-    <origin xyz="0 0 0" rpy="1.5708 1.5708 0"/>
+    <origin xyz="-0.01 -0.03 0" rpy="1.5708 1.5708 0"/>
     <geometry>
           <mesh filename="package://jax_description/meshes/front_right_thigh.stl"

Commit message: d

File: jax_ws/src/jax_description/urdf/jax.urdf.xacro (robot description, xacro)
@@ -61,10 +61,11 @@
   <limit lower="-0.6" upper="0.6" effort="1.0" velocity="1.0"/>
 </joint>
+<!-- x y z up and down -->
 <link name="front_right_thigh">
   <visual>
-    <origin xyz="-0.01 -0.03 0" rpy="1.5708 1.5708 0"/>
+    <origin xyz="0.06 0.01 0.03" rpy="1.5708 0 1.5708"/>
     <geometry>
           <mesh filename="package://jax_description/meshes/front_right_thigh.stl"
-          scale="1 1 1"/>
+          scale=".001 .001 .001"/>
   </geometry>
   </visual>

Commit message: meshes

File: jax_ws/src/jax_description/urdf/jax.urdf.xacro (robot description, xacro)
@@ -25,5 +25,5 @@
           scale="1 1 1"/>
   </geometry>
-  <material name="black"/>
+  <material name="white"/>
 </visual>
 <collision>
@@ -46,10 +46,10 @@
   <link name="front_right_hip">
     <visual>
-      <origin xyz="-0.01 0.02 -0.015" rpy="-1.5708 3.1416 -1.5708"/>
+      <origin xyz="0 -0.035 0.01" rpy="0 0 0"/>
       <geometry>
-        <mesh filename="package://jax_description/meshes/front_right_hip.stl"
-          scale="1 1 1"/>
+        <mesh filename="package://jax_description/meshes/right_hip.stl"
+          scale=".001 .001 .001"/>
       </geometry>
-      <material name="white"/>
+      <material name="black"/>
     </visual>
   </link>
@@ -57,16 +57,16 @@
   <parent link="base_link"/>
   <child link="front_right_hip"/>
-  <origin xyz="0.12 -0.08 0.0"/>
-  <axis xyz="1 0 0"/>
-  <limit lower="-0.6" upper="0.6" effort="1.0" velocity="1.0"/>
-</joint>
-<!-- x y z up and down -->
+  <origin xyz="0.11 -0.06 -0.01"/>
+  <axis xyz="1 0 0"/>
+  <limit lower="-0.6" upper="0.6" effort="1.0" velocity="1.0"/>
+</joint>
 <link name="front_right_thigh">
   <visual>
-    <origin xyz="0.06 0.01 0.03" rpy="1.5708 0 1.5708"/>
-    <geometry>
-          <mesh filename="package://jax_description/meshes/front_right_thigh.stl"
+    <origin xyz="0 -.038 0" rpy="0 0 0"/>
+    <geometry>
+          <mesh filename="package://jax_description/meshes/right_thigh.stl"
           scale=".001 .001 .001"/>
   </geometry>
+    <material name="white"/>
   </visual>
 </link>
@@ -74,14 +74,16 @@
     <parent link="front_right_hip"/>
     <child link="front_right_thigh"/>
-    <origin xyz="0 0 0"/>
+    <origin xyz="0 0 0.01"/>
     <axis xyz="0 -1 0"/>
-    <limit lower="-1.57" upper="1.57" effort="1.0" velocity="1.0"/>
+    <limit lower="-1.2" upper="1.2" effort="1.0" velocity="1.0"/>
   </joint>
   <link name="front_right_calf">
     <visual>
-      <origin xyz="0 0 -0.06"/>
+      <origin xyz="0 -0.048 0" rpy="0 0 0"/>
       <geometry>
-        <cylinder length="0.12" radius="0.012"/>
+        <mesh filename="package://jax_description/meshes/right_calf.stl"
+          scale=".001 .001 .001"/>
       </geometry>
+      <material name="black"/>
     </visual>
    </link>
@@ -89,13 +91,15 @@
   <parent link="front_right_thigh"/>
   <child link="front_right_calf"/>
-  <origin xyz="0 0 -0.12"/>
-  <axis xyz="0 1 0"/>
-  <limit lower="0.0" upper="1.57" effort="1.0" velocity="1.0"/>
+  <origin xyz="0 0 -0.13"/>
+  <axis xyz="0 -1 0"/>
+  <limit lower="0" upper="1.4" effort="1.0" velocity="1.0"/>
 </joint>
 <!-- FRONT LEFT LEG -->
 <link name="front_left_hip">
   <visual>
-    <geometry>
-      <cylinder length="0.05" radius="0.02"/>
+    <origin xyz="0 0.035 0.01" rpy="0 0 0"/>
+    <geometry>
+      <mesh filename="package://jax_description/meshes/left_hip.stl"
+            scale=".001 .001 .001"/>
     </geometry>
     <material name="black"/>
@@ -105,5 +109,5 @@
   <parent link="base_link"/>
   <child link="front_left_hip"/>
-  <origin xyz="0.12 0.08 0.0"/>
+  <origin xyz="0.11 0.06 -0.01"/>
   <axis xyz="1 0 0"/>
   <limit lower="-0.6" upper="0.6" effort="1.0" velocity="1.0"/>
@@ -111,8 +115,10 @@
 <link name="front_left_thigh">
   <visual>
-    <origin xyz="0 0 -0.06"/>
-    <geometry>
-      <cylinder length="0.12" radius="0.015"/>
-    </geometry>
+    <origin xyz="0 0.038 0" rpy="0 0 0"/>
+    <geometry>
+      <mesh filename="package://jax_description/meshes/left_thigh.stl"
+            scale=".001 .001 .001"/>
+    </geometry>
+    <material name="white"/>
   </visual>
 </link>
@@ -120,14 +126,16 @@
   <parent link="front_left_hip"/>
   <child link="front_left_thigh"/>
-  <origin xyz="0 0 0"/>
-  <axis xyz="0 1 0"/>
-  <limit lower="-1.57" upper="1.57" effort="1.0" velocity="1.0"/>
+  <origin xyz="0 0 0.01"/>
+  <axis xyz="0 -1 0"/>
+  <limit lower="-1.2" upper="1.2" effort="1.0" velocity="1.0"/>
 </joint>
 <link name="front_left_calf">
   <visual>
-    <origin xyz="0 0 -0.06"/>
-    <geometry>
-      <cylinder length="0.12" radius="0.012"/>
-    </geometry>
+    <origin xyz="0 0.048 0" rpy="0 0 0"/>
+    <geometry>
+      <mesh filename="package://jax_description/meshes/left_calf.stl"
+            scale=".001 .001 .001"/>
+    </geometry>
+    <material name="black"/>
   </visual>
 </link>
@@ -135,13 +143,15 @@
   <parent link="front_left_thigh"/>
   <child link="front_left_calf"/>
-  <origin xyz="0 0 -0.12"/>
-  <axis xyz="0 1 0"/>
-  <limit lower="0.0" upper="1.57" effort="1.0" velocity="1.0"/>
+  <origin xyz="0 0 -0.13"/>
+  <axis xyz="0 -1 0"/>
+  <limit lower="0" upper="1.4" effort="1.0" velocity="1.0"/>
 </joint>
 <!-- REAR RIGHT LEG -->
 <link name="rear_right_hip">
   <visual>
-    <geometry>
-      <cylinder length="0.05" radius="0.02"/>
+    <origin xyz="0 -0.035 0.01" rpy="0 0 0"/>
+    <geometry>
+      <mesh filename="package://jax_description/meshes/right_hip.stl"
+            scale=".001 .001 .001"/>
     </geometry>
     <material name="black"/>
@@ -151,5 +161,5 @@
   <parent link="base_link"/>
   <child link="rear_right_hip"/>
-  <origin xyz="-0.12 -0.08 0.0"/>
+  <origin xyz="-0.11 -0.06 -0.01"/>
   <axis xyz="1 0 0"/>
   <limit lower="-0.6" upper="0.6" effort="1.0" velocity="1.0"/>
@@ -157,8 +167,10 @@
 <link name="rear_right_thigh">
   <visual>
-    <origin xyz="0 0 -0.06"/>
-    <geometry>
-      <cylinder length="0.12" radius="0.015"/>
-    </geometry>
+    <origin xyz="0 -0.038 0" rpy="0 0 0"/>
+    <geometry>
+      <mesh filename="package://jax_description/meshes/right_thigh.stl"
+            scale=".001 .001 .001"/>
+    </geometry>
+    <material name="white"/>
   </visual>
 </link>
@@ -166,14 +178,16 @@
   <parent link="rear_right_hip"/>
   <child link="rear_right_thigh"/>
-  <origin xyz="0 0 0"/>
-  <axis xyz="0 -1 0"/>
-  <limit lower="-1.57" upper="1.57" effort="1.0" velocity="1.0"/>
+  <origin xyz="0 0 0.01"/>
+  <axis xyz="0 -1 0"/>
+  <limit lower="-1.2" upper="1.2" effort="1.0" velocity="1.0"/>
 </joint>
 <link name="rear_right_calf">
   <visual>
-    <origin xyz="0 0 -0.06"/>
-    <geometry>
-      <cylinder length="0.12" radius="0.012"/>
-    </geometry>
+    <origin xyz="0 -0.048 0" rpy="0 0 0"/>
+    <geometry>
+      <mesh filename="package://jax_description/meshes/right_calf.stl"
+            scale=".001 .001 .001"/>
+    </geometry>
+    <material name="black"/>
   </visual>
 </link>
@@ -181,13 +195,15 @@
   <parent link="rear_right_thigh"/>
   <child link="rear_right_calf"/>
-  <origin xyz="0 0 -0.12"/>
-  <axis xyz="0 1 0"/>
-  <limit lower="0.0" upper="1.57" effort="1.0" velocity="1.0"/>
+  <origin xyz="0 0 -0.13"/>
+  <axis xyz="0 -1 0"/>
+  <limit lower="0" upper="1.4" effort="1.0" velocity="1.0"/>
 </joint>
 <!-- REAR LEFT LEG -->
 <link name="rear_left_hip">
   <visual>
-    <geometry>
-      <cylinder length="0.05" radius="0.02"/>
+    <origin xyz="0 0.035 0.01" rpy="0 0 0"/>
+    <geometry>
+      <mesh filename="package://jax_description/meshes/left_hip.stl"
+            scale=".001 .001 .001"/>
     </geometry>
     <material name="black"/>
@@ -197,5 +213,5 @@
   <parent link="base_link"/>
   <child link="rear_left_hip"/>
-  <origin xyz="-0.12 0.08 0.0"/>
+  <origin xyz="-0.11 0.06 -0.01"/>
   <axis xyz="1 0 0"/>
   <limit lower="-0.6" upper="0.6" effort="1.0" velocity="1.0"/>
@@ -203,8 +219,10 @@
 <link name="rear_left_thigh">
   <visual>
-    <origin xyz="0 0 -0.06"/>
-    <geometry>
-      <cylinder length="0.12" radius="0.015"/>
-    </geometry>
+    <origin xyz="0 0.038 0" rpy="0 0 0"/>
+    <geometry>
+      <mesh filename="package://jax_description/meshes/left_thigh.stl"
+            scale=".001 .001 .001"/>
+    </geometry>
+    <material name="white"/>
   </visual>
 </link>
@@ -212,14 +230,16 @@
   <parent link="rear_left_hip"/>
   <child link="rear_left_thigh"/>
-  <origin xyz="0 0 0"/>
-  <axis xyz="0 1 0"/>
-  <limit lower="-1.57" upper="1.57" effort="1.0" velocity="1.0"/>
+  <origin xyz="0 0 0.01"/>
+  <axis xyz="0 -1 0"/>
+  <limit lower="-1.2" upper="1.2" effort="1.0" velocity="1.0"/>
 </joint>
 <link name="rear_left_calf">
   <visual>
-    <origin xyz="0 0 -0.06"/>
-    <geometry>
-      <cylinder length="0.12" radius="0.012"/>
-    </geometry>
+    <origin xyz="0 0.048 0" rpy="0 0 0"/>
+    <geometry>
+      <mesh filename="package://jax_description/meshes/left_calf.stl"
+            scale=".001 .001 .001"/>
+    </geometry>
+    <material name="black"/>
   </visual>
 </link>
@@ -227,7 +247,7 @@
   <parent link="rear_left_thigh"/>
   <child link="rear_left_calf"/>
-  <origin xyz="0 0 -0.12"/>
-  <axis xyz="0 1 0"/>
-  <limit lower="0.0" upper="1.57" effort="1.0" velocity="1.0"/>
+  <origin xyz="0 0 -0.13"/>
+  <axis xyz="0 -1 0"/>
+  <limit lower="0" upper="1.4" effort="1.0" velocity="1.0"/>
 </joint>
 </robot>

Commit message: vv

File: jax_ws/src/jax_description/urdf/jax.urdf.xacro (robot description, xacro)
@@ -14,14 +14,17 @@
     <color rgba="0.1 0.1 0.1 1.0"/>
   </material>
-  <material name="white">
+<material name="white">
   <color rgba="1 1 1 1"/>
+</material>
+<material name="debug">
+  <color rgba="1 0 0 0.4"/>
 </material>
 <!-- Base link -->
 <link name="base_link">
-  <visual>
+   <visual>
   <origin xyz="0 0 0" rpy="0 0 0"/>
   <geometry>
     <mesh filename="package://jax_description/meshes/base_link.stl"
-          scale="1 1 1"/>
+          scale=".001 .001 .001"/>
   </geometry>
   <material name="white"/>
@@ -31,5 +34,5 @@
   <geometry>
     <mesh filename="package://jax_description/meshes/base_collision.stl"
-          scale="1 1 1"/>
+          scale=".001 .001 .001"/>
   </geometry>
 </collision>
