Commit message: added collsion

File: jax_ws/src/jax_description/urdf/jax.urdf.xacro (robot description, xacro)
@@ -33,6 +33,5 @@
   <origin xyz="0 0 0" rpy="0 0 0"/>
   <geometry>
-    <mesh filename="package://jax_description/meshes/base_collision.stl"
-          scale=".001 .001 .001"/>
+    <box size="0.26 0.14 0.06"/>
   </geometry>
 </collision>
@@ -56,4 +55,18 @@
       <material name="black"/>
     </visual>
+        <collision>
+      <origin xyz="0 -0.02 0"/>
+    <geometry>
+      <sphere radius="0.025"/>
+    </geometry>
+  </collision>
+  <inertial>
+    <mass value="0.15"/>
+    <origin xyz="0 -0.02 0"/>
+    <inertia
+      ixx="0.0002" ixy="0" ixz="0"
+      iyy="0.0002" iyz="0"
+      izz="0.0002"/>
+  </inertial>
   </link>
 <joint name="front_right_hip_joint" type="revolute">
@@ -73,4 +86,18 @@
     <material name="white"/>
   </visual>
+ <collision>
+    <origin xyz="0 -.039 -0.065"/>
+    <geometry>
+      <cylinder radius="0.012" length="0.15"/>
+    </geometry>
+  </collision>
+  <inertial>
+    <mass value="0.35"/>
+    <origin xyz="0 -0.39 -0.065"/>
+    <inertia
+      ixx="0.001" ixy="0" ixz="0"
+      iyy="0.001" iyz="0"
+      izz="0.0003"/>
+  </inertial>
 </link>
   <joint name="front_right_thigh_joint" type="revolute">
@@ -90,4 +117,18 @@
       <material name="black"/>
     </visual>
+      <collision>
+    <origin xyz="0.05 -0.043 -0.045" rpy="0 -0.85 0"/>
+    <geometry>
+      <cylinder radius="0.012" length="0.13"/>
+    </geometry>
+  </collision>
+  <inertial>
+    <mass value="0.25"/>
+    <origin xyz="0.05 -0.043 -0.045" rpy="0 -0.85 0"/>
+    <inertia
+      ixx="0.0007" ixy="0" ixz="0"
+      iyy="0.0007" iyz="0"
+      izz="0.0002"/>
+  </inertial>
    </link>
   <joint name="front_right_knee_joint" type="revolute">
@@ -108,4 +149,18 @@
     </material>
   </visual>
+     <collision>
+    <origin xyz="0 0 0.005"/>
+    <geometry>
+      <sphere radius="0.010"/>
+    </geometry>
+  </collision>
+  <inertial>
+    <mass value="0.08"/>
+    <origin xyz="0 0 0.005"/>
+    <inertia
+      ixx="0.00005" ixy="0" ixz="0"
+      iyy="0.00005" iyz="0"
+      izz="0.00005"/>
+  </inertial>
   </link>
 <joint name="front_right_ankle_joint" type="fixed">
@@ -117,5 +172,5 @@
 <link name="front_left_hip">
   <visual>
-    <origin xyz="0 0.035 0.01" rpy="0 0 0"/>
+    <origin xyz="0 0.035 0.01"/>
     <geometry>
       <mesh filename="package://jax_description/meshes/left_hip.stl"
@@ -124,4 +179,17 @@
     <material name="black"/>
   </visual>
+  <collision>
+    <origin xyz="0 0.02 0"/>
+    <geometry>
+      <sphere radius="0.025"/>
+    </geometry>
+  </collision>
+  <inertial>
+    <mass value="0.15"/>
+    <origin xyz="0 0.02 0"/>
+    <inertia ixx="0.0002" ixy="0" ixz="0"
+             iyy="0.0002" iyz="0"
+             izz="0.0002"/>
+  </inertial>
 </link>
 <joint name="front_left_hip_joint" type="revolute">
@@ -134,5 +202,5 @@
 <link name="front_left_thigh">
   <visual>
-    <origin xyz="0 0.038 0" rpy="0 0 0"/>
+    <origin xyz="0 0.038 0"/>
     <geometry>
       <mesh filename="package://jax_description/meshes/left_thigh.stl"
@@ -141,4 +209,17 @@
     <material name="white"/>
   </visual>
+  <collision>
+    <origin xyz="0 0.039 -0.065"/>
+    <geometry>
+      <cylinder radius="0.012" length="0.15"/>
+    </geometry>
+  </collision>
+  <inertial>
+    <mass value="0.35"/>
+    <origin xyz="0 0.039 -0.065"/>
+    <inertia ixx="0.001" ixy="0" ixz="0"
+             iyy="0.001" iyz="0"
+             izz="0.0003"/>
+  </inertial>
 </link>
 <joint name="front_left_thigh_joint" type="revolute">
@@ -151,5 +232,5 @@
 <link name="front_left_calf">
   <visual>
-    <origin xyz="0 0.048 0" rpy="0 0 0"/>
+    <origin xyz="0 0.048 0"/>
     <geometry>
       <mesh filename="package://jax_description/meshes/left_calf.stl"
@@ -158,4 +239,17 @@
     <material name="black"/>
   </visual>
+  <collision>
+    <origin xyz="0.05 0.043 -0.045" rpy="0 -0.85 0"/>
+    <geometry>
+      <cylinder radius="0.012" length="0.13"/>
+    </geometry>
+  </collision>
+  <inertial>
+    <mass value="0.25"/>
+    <origin xyz="0.05 0.043 -0.045" rpy="0 -0.85 0"/>
+    <inertia ixx="0.0007" ixy="0" ixz="0"
+             iyy="0.0007" iyz="0"
+             izz="0.0002"/>
+  </inertial>
 </link>
 <joint name="front_left_knee_joint" type="revolute">
@@ -168,5 +262,4 @@
 <link name="front_left_foot">
   <visual>
-    <origin xyz="0 0 0" rpy="0 0 0"/>
     <geometry>
       <mesh filename="package://jax_description/meshes/foot.stl"
@@ -175,4 +268,17 @@
     <material name="black"/>
   </visual>
+  <collision>
+    <origin xyz="0 0 0.005"/>
+    <geometry>
+      <sphere radius="0.010"/>
+    </geometry>
+  </collision>
+  <inertial>
+    <mass value="0.08"/>
+    <origin xyz="0 0 0.005"/>
+    <inertia ixx="0.00005" ixy="0" ixz="0"
+             iyy="0.00005" iyz="0"
+             izz="0.00005"/>
+  </inertial>
 </link>
 <joint name="front_left_ankle_joint" type="fixed">
@@ -184,5 +290,5 @@
 <link name="rear_right_hip">
   <visual>
-    <origin xyz="0 -0.035 0.01" rpy="0 0 0"/>
+    <origin xyz="0 -0.035 0.01"/>
     <geometry>
       <mesh filename="package://jax_description/meshes/right_hip.stl"
@@ -191,4 +297,17 @@
     <material name="black"/>
   </visual>
+  <collision>
+    <origin xyz="0 -0.02 0"/>
+    <geometry>
+      <sphere radius="0.025"/>
+    </geometry>
+  </collision>
+  <inertial>
+    <mass value="0.15"/>
+    <origin xyz="0 -0.02 0"/>
+    <inertia ixx="0.0002" ixy="0" ixz="0"
+             iyy="0.0002" iyz="0"
+             izz="0.0002"/>
+  </inertial>
 </link>
 <joint name="rear_right_hip_joint" type="revolute">
@@ -201,5 +320,5 @@
 <link name="rear_right_thigh">
   <visual>
-    <origin xyz="0 -0.038 0" rpy="0 0 0"/>
+    <origin xyz="0 -0.038 0"/>
     <geometry>
       <mesh filename="package://jax_description/meshes/right_thigh.stl"
@@ -208,4 +327,17 @@
     <material name="white"/>
   </visual>
+  <collision>
+    <origin xyz="0 -0.039 -0.065"/>
+    <geometry>
+      <cylinder radius="0.012" length="0.15"/>
+    </geometry>
+  </collision>
+  <inertial>
+    <mass value="0.35"/>
+    <origin xyz="0 -0.039 -0.065"/>
+    <inertia ixx="0.001" ixy="0" ixz="0"
+             iyy="0.001" iyz="0"
+             izz="0.0003"/>
+  </inertial>
 </link>
 <joint name="rear_right_thigh_joint" type="revolute">
@@ -218,5 +350,5 @@
 <link name="rear_right_calf">
   <visual>
-    <origin xyz="0 -0.048 0" rpy="0 0 0"/>
+    <origin xyz="0 -0.048 0"/>
     <geometry>
       <mesh filename="package://jax_description/meshes/right_calf.stl"
@@ -225,4 +357,17 @@
     <material name="black"/>
   </visual>
+  <collision>
+    <origin xyz="0.05 -0.043 -0.045" rpy="0 -0.85 0"/>
+    <geometry>
+      <cylinder radius="0.012" length="0.13"/>
+    </geometry>
+  </collision>
+  <inertial>
+    <mass value="0.25"/>
+    <origin xyz="0.05 -0.043 -0.045" rpy="0 -0.85 0"/>
+    <inertia ixx="0.0007" ixy="0" ixz="0"
+             iyy="0.0007" iyz="0"
+             izz="0.0002"/>
+  </inertial>
 </link>
 <joint name="rear_right_knee_joint" type="revolute">
@@ -242,4 +387,18 @@
     <material name="black"/>
   </visual>
+  <collision>
+    <origin xyz="0 0 0.005"/>
+    <geometry>
+      <sphere radius="0.010"/>
+    </geometry>
+  </collision>
+  <inertial>
+    <mass value="0.08"/>
+    <origin xyz="0 0 0.005"/>
+    <inertia
+      ixx="0.00005" ixy="0" ixz="0"
+      iyy="0.00005" iyz="0"
+      izz="0.00005"/>
+  </inertial>
 </link>
 <joint name="rear_right_ankle_joint" type="fixed">
@@ -251,5 +410,5 @@
 <link name="rear_left_hip">
   <visual>
-    <origin xyz="0 0.035 0.01" rpy="0 0 0"/>
+    <origin xyz="0 0.035 0.01"/>
     <geometry>
       <mesh filename="package://jax_description/meshes/left_hip.stl"
@@ -258,4 +417,18 @@
     <material name="black"/>
   </visual>
+  <collision>
+    <origin xyz="0 0.02 0"/>
+    <geometry>
+      <sphere radius="0.025"/>
+    </geometry>
+  </collision>
+  <inertial>
+    <mass value="0.15"/>
+    <origin xyz="0 0.02 0"/>
+    <inertia
+      ixx="0.0002" ixy="0" ixz="0"
+      iyy="0.0002" iyz="0"
+      izz="0.0002"/>
+  </inertial>
 </link>
 <joint name="rear_left_hip_joint" type="revolute">
@@ -268,5 +441,5 @@
 <link name="rear_left_thigh">
   <visual>
-    <origin xyz="0 0.038 0" rpy="0 0 0"/>
+    <origin xyz="0 0.038 0"/>
     <geometry>
       <mesh filename="package://jax_description/meshes/left_thigh.stl"
@@ -275,4 +448,18 @@
     <material name="white"/>
   </visual>
+  <collision>
+    <origin xyz="0 0.039 -0.065"/>
+    <geometry>
+      <cylinder radius="0.012" length="0.15"/>
+    </geometry>
+  </collision>
+  <inertial>
+    <mass value="0.35"/>
+    <origin xyz="0 0.039 -0.065"/>
+    <inertia
+      ixx="0.001" ixy="0" ixz="0"
+      iyy="0.001" iyz="0"
+      izz="0.0003"/>
+  </inertial>
 </link>
 <joint name="rear_left_thigh_joint" type="revolute">
@@ -285,5 +472,5 @@
 <link name="rear_left_calf">
   <visual>
-    <origin xyz="0 0.048 0" rpy="0 0 0"/>
+    <origin xyz="0 0.048 0"/>
     <geometry>
       <mesh filename="package://jax_description/meshes/left_calf.stl"
@@ -292,4 +479,18 @@
     <material name="black"/>
   </visual>
+  <collision>
+    <origin xyz="0.05 0.043 -0.045" rpy="0 -0.85 0"/>
+    <geometry>
+      <cylinder radius="0.012" length="0.13"/>
+    </geometry>
+  </collision>
+  <inertial>
+    <mass value="0.25"/>
+    <origin xyz="0.05 0.043 -0.045" rpy="0 -0.85 0"/>
+    <inertia
+      ixx="0.0007" ixy="0" ixz="0"
+      iyy="0.0007" iyz="0"
+      izz="0.0002"/>
+  </inertial>
 </link>
 <joint name="rear_left_knee_joint" type="revolute">
@@ -302,5 +503,4 @@
 <link name="rear_left_foot">
   <visual>
-    <origin xyz="0 0 0" rpy="0 0 0"/>
     <geometry>
       <mesh filename="package://jax_description/meshes/foot.stl"
@@ -309,4 +509,18 @@
     <material name="black"/>
   </visual>
+  <collision>
+    <origin xyz="0 0 0.005"/>
+    <geometry>
+      <sphere radius="0.010"/>
+    </geometry>
+  </collision>
+  <inertial>
+    <mass value="0.08"/>
+    <origin xyz="0 0 0.005"/>
+    <inertia
+      ixx="0.00005" ixy="0" ixz="0"
+      iyy="0.00005" iyz="0"
+      izz="0.00005"/>
+  </inertial>
 </link>
 <joint name="rear_left_ankle_joint" type="fixed">

Commit message: fix

File: jax_ws/src/jax_description/urdf/jax.urdf.xacro (robot description, xacro)
@@ -23,17 +23,17 @@
 <link name="base_link">
    <visual>
-  <origin xyz="0 0 0" rpy="0 0 0"/>
-  <geometry>
-    <mesh filename="package://jax_description/meshes/base_link.stl"
+    <origin xyz="0 0 0" rpy="0 0 0"/>
+      <geometry>
+        <mesh filename="package://jax_description/meshes/base_link.stl"
           scale="1 1 1"/>
-  </geometry>
-  <material name="white"/>
-</visual>
-<collision>
+     </geometry>
+    <material name="white"/>
+    </visual>
+  <collision>
   <origin xyz="0 0 0" rpy="0 0 0"/>
   <geometry>
     <box size="0.26 0.14 0.06"/>
   </geometry>
-</collision>
+  </collision>
   <inertial>
     <mass value="3.0"/>
@@ -55,18 +55,18 @@
       <material name="black"/>
     </visual>
-        <collision>
+     <collision>
       <origin xyz="0 -0.02 0"/>
-    <geometry>
+     <geometry>
       <sphere radius="0.025"/>
-    </geometry>
-  </collision>
-  <inertial>
-    <mass value="0.15"/>
-    <origin xyz="0 -0.02 0"/>
-    <inertia
+     </geometry>
+     </collision>
+    <inertial>
+      <mass value="0.15"/>
+      <origin xyz="0 -0.02 0"/>
+      <inertia
       ixx="0.0002" ixy="0" ixz="0"
       iyy="0.0002" iyz="0"
       izz="0.0002"/>
-  </inertial>
+    </inertial>
   </link>
 <joint name="front_right_hip_joint" type="revolute">
@@ -75,5 +75,6 @@
   <origin xyz="0.11 -0.06 -0.01"/>
   <axis xyz="1 0 0"/>
-  <limit lower="-0.6" upper="0.6" effort="1.0" velocity="1.0"/>
+  <limit lower="-0.6" upper="0.6" effort="2.0" velocity="1.5"/>
+  <dynamics damping="0.5" friction="0.0"/>
 </joint>
 <link name="front_right_thigh">
@@ -83,8 +84,8 @@
           <mesh filename="package://jax_description/meshes/right_thigh.stl"
           scale=".001 .001 .001"/>
-  </geometry>
+    </geometry>
     <material name="white"/>
   </visual>
- <collision>
+  <collision>
     <origin xyz="0 -.039 -0.065"/>
     <geometry>
@@ -106,5 +107,6 @@
     <origin xyz="0 0 0.01"/>
     <axis xyz="0 -1 0"/>
-    <limit lower="-1.2" upper="1.2" effort="1.0" velocity="1.0"/>
+    <limit lower="-1.2" upper="1.2" effort="3.0" velocity="2.0"/>
+    <dynamics damping="0.7" friction="0.0"/>
   </joint>
   <link name="front_right_calf">
@@ -117,19 +119,19 @@
       <material name="black"/>
     </visual>
-      <collision>
-    <origin xyz="0.05 -0.043 -0.045" rpy="0 -0.85 0"/>
-    <geometry>
-      <cylinder radius="0.012" length="0.13"/>
-    </geometry>
-  </collision>
-  <inertial>
-    <mass value="0.25"/>
-    <origin xyz="0.05 -0.043 -0.045" rpy="0 -0.85 0"/>
-    <inertia
+    <collision>
+      <origin xyz="0.05 -0.043 -0.045" rpy="0 -0.85 0"/>
+      <geometry>
+        <cylinder radius="0.012" length="0.13"/>
+      </geometry>
+    </collision>
+    <inertial>
+      <mass value="0.25"/>
+      <origin xyz="0.05 -0.043 -0.045" rpy="0 -0.85 0"/>
+      <inertia
       ixx="0.0007" ixy="0" ixz="0"
       iyy="0.0007" iyz="0"
       izz="0.0002"/>
-  </inertial>
-   </link>
+    </inertial>
+  </link>
   <joint name="front_right_knee_joint" type="revolute">
   <parent link="front_right_thigh"/>
@@ -137,8 +139,9 @@
   <origin xyz="0 0 -0.13"/>
   <axis xyz="0 -1 0"/>
-  <limit lower="0" upper="1.4" effort="1.0" velocity="1.0"/>
+  <limit lower="0" upper="1.4" effort="4.0" velocity="2.5"/>
+  <dynamics damping="0.9" friction="0.0"/>
 </joint>
 <link name="front_right_foot">
-    <visual>
+  <visual>
     <origin xyz="0 0 0" rpy="0 0 0"/>
     <geometry>
@@ -149,5 +152,5 @@
     </material>
   </visual>
-     <collision>
+  <collision>
     <origin xyz="0 0 0.005"/>
     <geometry>
@@ -163,5 +166,5 @@
       izz="0.00005"/>
   </inertial>
-  </link>
+</link>
 <joint name="front_right_ankle_joint" type="fixed">
   <parent link="front_right_calf"/>
@@ -169,4 +172,10 @@
   <origin xyz="0.095 -0.044 -0.1" rpy="0 0 0"/>
 </joint>
+<gazebo reference="front_right_foot">
+  <mu1>1.2</mu1>
+  <mu2>1.2</mu2>
+  <kp>100000</kp>
+  <kd>100</kd>
+</gazebo>
 <!-- FRONT LEFT LEG -->
 <link name="front_left_hip">
@@ -198,5 +207,6 @@
   <origin xyz="0.11 0.06 -0.01"/>
   <axis xyz="1 0 0"/>
-  <limit lower="-0.6" upper="0.6" effort="1.0" velocity="1.0"/>
+  <limit lower="-0.6" upper="0.6" effort="2.0" velocity="1.5"/>
+  <dynamics damping="0.5" friction="0.0"/>
 </joint>
 <link name="front_left_thigh">
@@ -228,5 +238,6 @@
   <origin xyz="0 0 0.01"/>
   <axis xyz="0 -1 0"/>
-  <limit lower="-1.2" upper="1.2" effort="1.0" velocity="1.0"/>
+  <limit lower="-1.2" upper="1.2" effort="3.0" velocity="2.0"/>
+  <dynamics damping="0.7" friction="0.0"/>
 </joint>
 <link name="front_left_calf">
@@ -258,5 +269,6 @@
   <origin xyz="0 0 -0.13"/>
   <axis xyz="0 -1 0"/>
-  <limit lower="0" upper="1.4" effort="1.0" velocity="1.0"/>
+  <limit lower="0" upper="1.4" effort="4.0" velocity="2.5"/>
+  <dynamics damping="0.9" friction="0.0"/>
 </joint>
 <link name="front_left_foot">
@@ -287,4 +299,10 @@
   <origin xyz="0.095 0.044 -0.1" rpy="0 0 0"/>
 </joint>
+<gazebo reference="front_left_foot">
+  <mu1>1.2</mu1>
+  <mu2>1.2</mu2>
+  <kp>100000</kp>
+  <kd>100</kd>
+</gazebo>
 <!-- REAR RIGHT LEG -->
 <link name="rear_right_hip">
@@ -316,5 +334,6 @@
   <origin xyz="-0.11 -0.06 -0.01"/>
   <axis xyz="1 0 0"/>
-  <limit lower="-0.6" upper="0.6" effort="1.0" velocity="1.0"/>
+  <limit lower="-0.6" upper="0.6" effort="2.0" velocity="1.5"/>
+  <dynamics damping="0.5" friction="0.0"/>
 </joint>
 <link name="rear_right_thigh">
@@ -346,5 +365,6 @@
   <origin xyz="0 0 0.01"/>
   <axis xyz="0 -1 0"/>
-  <limit lower="-1.2" upper="1.2" effort="1.0" velocity="1.0"/>
+  <limit lower="-1.2" upper="1.2" effort="3.0" velocity="2.0"/>
+  <dynamics damping="0.7" friction="0.0"/>
 </joint>
 <link name="rear_right_calf">
@@ -376,5 +396,6 @@
   <origin xyz="0 0 -0.13"/>
   <axis xyz="0 -1 0"/>
-  <limit lower="0" upper="1.4" effort="1.0" velocity="1.0"/>
+  <limit lower="0" upper="1.4" effort="4.0" velocity="2.5"/>
+  <dynamics damping="0.9" friction="0.0"/>
 </joint>
 <link name="rear_right_foot">
@@ -407,4 +428,10 @@
   <origin xyz="0.095 -0.044 -0.1" rpy="0 0 0"/>
 </joint>
+<gazebo reference="rear_right_foot">
+  <mu1>1.2</mu1>
+  <mu2>1.2</mu2>
+  <kp>100000</kp>
+  <kd>100</kd>
+</gazebo>
 <!-- REAR LEFT LEG -->
 <link name="rear_left_hip">
@@ -437,5 +464,6 @@
   <origin xyz="-0.11 0.06 -0.01"/>
   <axis xyz="1 0 0"/>
-  <limit lower="-0.6" upper="0.6" effort="1.0" velocity="1.0"/>
+  <limit lower="-0.6" upper="0.6" effort="2.0" velocity="1.5"/>
+  <dynamics damping="0.5" friction="0.0"/>
 </joint>
 <link name="rear_left_thigh">
@@ -468,5 +496,6 @@
   <origin xyz="0 0 0.01"/>
   <axis xyz="0 -1 0"/>
-  <limit lower="-1.2" upper="1.2" effort="1.0" velocity="1.0"/>
+  <limit lower="-1.2" upper="1.2" effort="3.0" velocity="2.0"/>
+  <dynamics damping="0.7" friction="0.0"/>
 </joint>
 <link name="rear_left_calf">
@@ -499,5 +528,6 @@
   <origin xyz="0 0 -0.13"/>
   <axis xyz="0 -1 0"/>
-  <limit lower="0" upper="1.4" effort="1.0" velocity="1.0"/>
+  <limit lower="0" upper="1.4" effort="4.0" velocity="2.5"/>
+  <dynamics damping="0.9" friction="0.0"/>
 </joint>
 <link name="rear_left_foot">
@@ -529,3 +559,9 @@
   <origin xyz="0.095 0.044 -0.1" rpy="0 0 0"/>
 </joint>
+<gazebo reference="rear_left_foot">
+  <mu1>1.2</mu1>
+  <mu2>1.2</mu2>
+  <kp>100000</kp>
+  <kd>100</kd>
+</gazebo>
 </robot>
