Commit message: Clean repo: ignore ROS build and log artifacts

File: install/jax_description/share/jax_description/urdf/jax.urdf.xacro (robot description, xacro)
@@ -24,6 +24,5 @@
 <collision>
   <geometry>
-    <mesh filename="package://jax_description/meshes/base_link.stl"
-            scale="0.001 0.001 0.001"/>
+    <box size="0.25 0.15 0.05"/>
   </geometry>
 </collision>

Commit message: Ignore colcon build artifacts

File: install/jax_description/share/jax_description/urdf/jax.urdf.xacro (robot description, xacro)
@@ -1,222 +1 @@
-<?xml version="1.0"?>
-<robot name="jax"
-xmlns:xacro="http://www.ros.org/wiki/xacro">
-  <!-- World link -->
-  <link name="world"/>
-  <!-- Fixed joint to base -->
-  <joint name="world_to_base" type="fixed">
-    <parent link="world"/>
-    <child link="base_link"/>
-    <origin xyz="0 0 0" rpy="0 0 0"/>
-  </joint>
-  <!-- Materials -->
-<material name="black">
-    <color rgba="0.1 0.1 0.1 1.0"/>
-  </material>
-<!-- Base link -->
-<link name="base_link">
-    <visual>
-      <geometry>
-          <box size="0.25 0.15 0.05"/>
-      </geometry>
-      <material name="black"/>
-    </visual>
-<collision>
-  <geometry>
-    <box size="0.25 0.15 0.05"/>
-  </geometry>
-</collision>
-    <inertial>
-      <mass value="3.0"/>
-      <origin xyz="0 0 0"/>
-      <inertia
-        ixx="0.02" ixy="0.0" ixz="0.0"
-        iyy="0.04" iyz="0.0"
-        izz="0.05"/>
-    </inertial>
-</link>
-  <!-- FRONT RIGHT LEG -->
-  <link name="front_right_hip">
-    <visual>
-      <geometry>
-        <cylinder length="0.05" radius="0.02"/>
-      </geometry>
-      <material name="black"/>
-    </visual>
-  </link>
-<joint name="front_right_hip_joint" type="revolute">
-  <parent link="base_link"/>
-  <child link="front_right_hip"/>
-  <origin xyz="0.12 -0.08 0.0"/>
-  <axis xyz="1 0 0"/>
-  <limit lower="-0.6" upper="0.6" effort="1.0" velocity="1.0"/>
-</joint>
-<link name="front_right_thigh">
-  <visual>
-    <origin xyz="0 0 -0.06"/>
-    <geometry>
-         <cylinder length="0.12" radius="0.015"/>
-  </geometry>
-  </visual>
-</link>
-  <joint name="front_right_thigh_joint" type="revolute">
-    <parent link="front_right_hip"/>
-    <child link="front_right_thigh"/>
-    <origin xyz="0 0 0"/>
-    <axis xyz="0 -1 0"/>
-    <limit lower="-1.57" upper="1.57" effort="1.0" velocity="1.0"/>
-  </joint>
-  <link name="front_right_calf">
-    <visual>
-      <origin xyz="0 0 -0.06"/>
-      <geometry>
-        <cylinder length="0.12" radius="0.012"/>
-      </geometry>
-    </visual>
-   </link>
-  <joint name="front_right_knee_joint" type="revolute">
-  <parent link="front_right_thigh"/>
-  <child link="front_right_calf"/>
-  <origin xyz="0 0 -0.12"/>
-  <axis xyz="0 1 0"/>
-  <limit lower="0.0" upper="1.57" effort="1.0" velocity="1.0"/>
-</joint>
-<!-- FRONT LEFT LEG -->
-<link name="front_left_hip">
-  <visual>
-    <geometry>
-      <cylinder length="0.05" radius="0.02"/>
-    </geometry>
-    <material name="black"/>
-  </visual>
-</link>
-<joint name="front_left_hip_joint" type="revolute">
-  <parent link="base_link"/>
-  <child link="front_left_hip"/>
-  <origin xyz="0.12 0.08 0.0"/>
-  <axis xyz="1 0 0"/>
-  <limit lower="-0.6" upper="0.6" effort="1.0" velocity="1.0"/>
-</joint>
-<link name="front_left_thigh">
-  <visual>
-    <origin xyz="0 0 -0.06"/>
-    <geometry>
-      <cylinder length="0.12" radius="0.015"/>
-    </geometry>
-  </visual>
-</link>
-<joint name="front_left_thigh_joint" type="revolute">
-  <parent link="front_left_hip"/>
-  <child link="front_left_thigh"/>
-  <origin xyz="0 0 0"/>
-  <axis xyz="0 1 0"/>
-  <limit lower="-1.57" upper="1.57" effort="1.0" velocity="1.0"/>
-</joint>
-<link name="front_left_calf">
-  <visual>
-    <origin xyz="0 0 -0.06"/>
-    <geometry>
-      <cylinder length="0.12" radius="0.012"/>
-    </geometry>
-  </visual>
-</link>
-<joint name="front_left_knee_joint" type="revolute">
-  <parent link="front_left_thigh"/>
-  <child link="front_left_calf"/>
-  <origin xyz="0 0 -0.12"/>
-  <axis xyz="0 1 0"/>
-  <limit lower="0.0" upper="1.57" effort="1.0" velocity="1.0"/>
-</joint>
-<!-- REAR RIGHT LEG -->
-<link name="rear_right_hip">
-  <visual>
-    <geometry>
-      <cylinder length="0.05" radius="0.02"/>
-    </geometry>
-    <material name="black"/>
-  </visual>
-</link>
-<joint name="rear_right_hip_joint" type="revolute">
-  <parent link="base_link"/>
-  <child link="rear_right_hip"/>
-  <origin xyz="-0.12 -0.08 0.0"/>
-  <axis xyz="1 0 0"/>
-  <limit lower="-0.6" upper="0.6" effort="1.0" velocity="1.0"/>
-</joint>
-<link name="rear_right_thigh">
-  <visual>
-    <origin xyz="0 0 -0.06"/>
-    <geometry>
-      <cylinder length="0.12" radius="0.015"/>
-    </geometry>
-  </visual>
-</link>
-<joint name="rear_right_thigh_joint" type="revolute">
-  <parent link="rear_right_hip"/>
-  <child link="rear_right_thigh"/>
-  <origin xyz="0 0 0"/>
-  <axis xyz="0 -1 0"/>
-  <limit lower="-1.57" upper="1.57" effort="1.0" velocity="1.0"/>
-</joint>
-<link name="rear_right_calf">
-  <visual>
-    <origin xyz="0 0 -0.06"/>
-    <geometry>
-      <cylinder length="0.12" radius="0.012"/>
-    </geometry>
-  </visual>
-</link>
-<joint name="rear_right_knee_joint" type="revolute">
-  <parent link="rear_right_thigh"/>
-  <child link="rear_right_calf"/>
-  <origin xyz="0 0 -0.12"/>
-  <axis xyz="0 1 0"/>
-  <limit lower="0.0" upper="1.57" effort="1.0" velocity="1.0"/>
-</joint>
-<!-- REAR LEFT LEG -->
-<link name="rear_left_hip">
-  <visual>
-    <geometry>
-      <cylinder length="0.05" radius="0.02"/>
-    </geometry>
-    <material name="black"/>
-  </visual>
-</link>
-<joint name="rear_left_hip_joint" type="revolute">
-  <parent link="base_link"/>
-  <child link="rear_left_hip"/>
-  <origin xyz="-0.12 0.08 0.0"/>
-  <axis xyz="1 0 0"/>
-  <limit lower="-0.6" upper="0.6" effort="1.0" velocity="1.0"/>
-</joint>
-<link name="rear_left_thigh">
-  <visual>
-    <origin xyz="0 0 -0.06"/>
-    <geometry>
-      <cylinder length="0.12" radius="0.015"/>
-    </geometry>
-  </visual>
-</link>
-<joint name="rear_left_thigh_joint" type="revolute">
-  <parent link="rear_left_hip"/>
-  <child link="rear_left_thigh"/>
-  <origin xyz="0 0 0"/>
-  <axis xyz="0 1 0"/>
-  <limit lower="-1.57" upper="1.57" effort="1.0" velocity="1.0"/>
-</joint>
-<link name="rear_left_calf">
-  <visual>
-    <origin xyz="0 0 -0.06"/>
-    <geometry>
-      <cylinder length="0.12" radius="0.012"/>
-    </geometry>
-  </visual>
-</link>
-<joint name="rear_left_knee_joint" type="revolute">
-  <parent link="rear_left_thigh"/>
-  <child link="rear_left_calf"/>
-  <origin xyz="0 0 -0.12"/>
-  <axis xyz="0 1 0"/>
-  <limit lower="0.0" upper="1.57" effort="1.0" velocity="1.0"/>
-</joint>
-</robot>
+/home/tdp378/Jax_Quadruped_ros2/build/jax_description/urdf/jax.urdf.xacro

File: jax_ws/src/jax_description/urdf/jax.urdf.xacro (robot description, xacro)
@@ -8,5 +8,5 @@
     <parent link="world"/>
     <child link="base_link"/>
-    <origin xyz="0 0 0" rpy="0 0 0"/>
+    <origin xyz="0 0 0.23" rpy="0 0 0"/>
   </joint>
   <!-- Materials -->
@@ -26,5 +26,5 @@
   <geometry>
     <mesh filename="package://jax_description/meshes/base_link.stl"
-          scale=".1 .1 .1"/>
+          scale="1 1 1"/>
   </geometry>
   <material name="white"/>
@@ -98,4 +98,20 @@
   <limit lower="0" upper="1.4" effort="1.0" velocity="1.0"/>
 </joint>
+<link name="front_right_foot">
+    <visual>
+    <origin xyz="0 0 0" rpy="0 0 0"/>
+    <geometry>
+      <mesh filename="package://jax_description/meshes/foot.stl"
+            scale=".001 .001 .001"/>
+    </geometry>
+    <material name="black">
+    </material>
+  </visual>
+  </link>
+<joint name="front_right_ankle_joint" type="fixed">
+  <parent link="front_right_calf"/>
+  <child link="front_right_foot"/>
+  <origin xyz="0.095 -0.044 -0.1" rpy="0 0 0"/>
+</joint>
 <!-- FRONT LEFT LEG -->
 <link name="front_left_hip">
@@ -150,4 +166,19 @@
   <limit lower="0" upper="1.4" effort="1.0" velocity="1.0"/>
 </joint>
+<link name="front_left_foot">
+  <visual>
+    <origin xyz="0 0 0" rpy="0 0 0"/>
+    <geometry>
+      <mesh filename="package://jax_description/meshes/foot.stl"
+            scale=".001 .001 .001"/>
+    </geometry>
+    <material name="black"/>
+  </visual>
+</link>
+<joint name="front_left_ankle_joint" type="fixed">
+  <parent link="front_left_calf"/>
+  <child link="front_left_foot"/>
+  <origin xyz="0.095 0.044 -0.1" rpy="0 0 0"/>
+</joint>
 <!-- REAR RIGHT LEG -->
 <link name="rear_right_hip">
@@ -202,4 +233,19 @@
   <limit lower="0" upper="1.4" effort="1.0" velocity="1.0"/>
 </joint>
+<link name="rear_right_foot">
+  <visual>
+    <origin xyz="0 0 0" rpy="0 0 0"/>
+    <geometry>
+      <mesh filename="package://jax_description/meshes/foot.stl"
+            scale=".001 .001 .001"/>
+    </geometry>
+    <material name="black"/>
+  </visual>
+</link>
+<joint name="rear_right_ankle_joint" type="fixed">
+  <parent link="rear_right_calf"/>
+  <child link="rear_right_foot"/>
+  <origin xyz="0.095 -0.044 -0.1" rpy="0 0 0"/>
+</joint>
 <!-- REAR LEFT LEG -->
 <link name="rear_left_hip">
@@ -254,3 +300,18 @@
   <limit lower="0" upper="1.4" effort="1.0" velocity="1.0"/>
 </joint>
+<link name="rear_left_foot">
+  <visual>
+    <origin xyz="0 0 0" rpy="0 0 0"/>
+    <geometry>
+      <mesh filename="package://jax_description/meshes/foot.stl"
+            scale=".001 .001 .001"/>
+    </geometry>
+    <material name="black"/>
+  </visual>
+</link>
+<joint name="rear_left_ankle_joint" type="fixed">
+  <parent link="rear_left_calf"/>
+  <child link="rear_left_foot"/>
+  <origin xyz="0.095 0.044 -0.1" rpy="0 0 0"/>
+</joint>
 </robot>
